Commit message: WIP - debugging grasp pose

File: src/ndf_robot/descriptions/hanging/table/table_tmp.urdf (robot description, URDF)
Before this commit: robot table.urdf, 2 links, 1 joints
Links:
- link shelf: geometry collision mesh filename=shelf_back.stl scale=0.75 0.75 0.5; visual mesh filename=shelf_back.stl scale=0.75 0.75 0.5
