Commit message: debugging ndf

File: src/rndf_robot/descriptions/hanging/table/table_peg_manual.urdf (robot description, URDF)
Before this commit: robot table.urdf, 2 links, 1 joints
Joints:
- joint table2peg: origin xyz=0.27 -0.09 0.9715 rpy=0 0 3.1415 -> xyz=0.27 -0.09 1.001 rpy=0 0 3.1415

File: src/rndf_robot/descriptions/hanging/table/table_shelf_manual.urdf (robot description, URDF)
Before this commit: robot table.urdf, 2 links, 1 joints
Links:
- link shelf: geometry collision mesh filename=shelf_back.obj scale=0.75 0.75 0.5; visual mesh filename=shelf_back.obj scale=0.75 0.75 0.5
